File: hardware/board/board/board.sch (EAGLE design)
At the start: 2 parts, among them M1 WIRELESS-NRF24L01

Commit message: added schematic and board files
Parts:
- added C1, C2: 10 uF, rcl:C-EUC0805
- added LED1: (no value), led:LED5MM
- added R1: (no value), rcl:R-EU_R0805
- added X1: MAB7SH, con-hirschmann:MAB7SH
Connections:
- new net 3V3: C1.2, M1.VCC
- new net GND: ARDUINO_NANO1.GND@1, ARDUINO_NANO1.GND@2, C1.1, C2.2, LED1.C, M1.GND, X1.7
- new net N$1: ARDUINO_NANO1.D13, M1.SCK
- new net N$10: ARDUINO_NANO1.D4, X1.1
- new net N$11: ARDUINO_NANO1.A1, X1.5
- new net N$12: ARDUINO_NANO1.D2, X1.4
- new net N$2: ARDUINO_NANO1.D12, M1.MISO
- new net N$3: ARDUINO_NANO1.D11, M1.MOSI
- new net N$4: ARDUINO_NANO1.D10, M1.CSN
- new net N$5: ARDUINO_NANO1.D9, M1.CE
- new net N$6: LED1.A, R1.2
- new net N$7: ARDUINO_NANO1.D3, R1.1
- new net N$8: ARDUINO_NANO1.D6, X1.6
- new net N$9: ARDUINO_NANO1.A2, X1.3
- new net VIN: C2.1, X1.2
Other:
- moved on the sheet: ARDUINO_NANO1, M1

Commit message: value update
Parts:
- R1: value (none) -> 220
Changed lines of the file:
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@@
 <part name="LED1" library="led" library_urn="urn:adsk.eagle:library:259" deviceset="LED" device="5MM" package3d_urn="urn:adsk.eagle:package:15799/2"/>
 <part name="C1" library="rcl" library_urn="urn:adsk.eagle:library:334" deviceset="C-EU" device="C0805" package3d_urn="urn:adsk.eagle:package:23617/2" value="10 uF"/>
-<part name="R1" library="rcl" library_urn="urn:adsk.eagle:library:334" deviceset="R-EU_" device="R0805" package3d_urn="urn:adsk.eagle:package:23553/2"/>
+<part name="R1" library="rcl" library_urn="urn:adsk.eagle:library:334" deviceset="R-EU_" device="R0805" package3d_urn="urn:adsk.eagle:package:23553/2" value="220"/>
 <part name="GND4" library="supply1" library_urn="urn:adsk.eagle:library:371" deviceset="GND" device=""/>
 <part name="X1" library="con-hirschmann" library_urn="urn:adsk.eagle:library:153" deviceset="MAB7SH" device="" package3d_urn="urn:adsk.eagle:package:7450/1"/>

Commit message: connected 3V3 radio line to the aruino nano
Connections:
- net 3V3: now also ARDUINO_NANO1.3V3
Changed lines of the file:
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@@
 <label x="129.54" y="78.74" size="1.778" layer="95"/>
+</segment>
+<segment>
+<pinref part="ARDUINO_NANO1" gate="G$1" pin="3V3"/>
+<wire x1="30.48" y1="88.9" x2="25.4" y2="88.9" width="0.1524" layer="91"/>
+<label x="20.32" y="88.9" size="1.778" layer="95"/>
 </segment>
 </net>
